Commit message: lidar, readme, joy added

File: four_w_amr/urdf/four_w_amr.urdf (robot description, URDF)
Before this commit: robot four_w_amr, 8 links, 7 joints
Joints:
- joint back_left_joint: axis 0 0 -1 -> 0 1 0; origin xyz=-0.09 0.12514 -0.0092692 rpy=1.5708 0 0 -> xyz=-0.09 0.12514 -0.0092692 rpy=0 0 0
- joint back_right_joint: axis 0 0 1 -> 0 1 0; origin xyz=-0.09 -0.12514 -0.0092692 rpy=1.5708 0 0 -> xyz=-0.09 -0.12514 -0.0092692 rpy=0 0 0
- joint front_left_joint: axis 0 0 -1 -> 0 1 0; origin xyz=0.09 0.12514 -0.0092692 rpy=1.5708 0 0 -> xyz=0.09 0.12514 -0.0092692 rpy=0 0 0
- joint front_right_joint: axis 0 0 1 -> 0 1 0; origin xyz=0.09 -0.12514 -0.0092692 rpy=1.5708 0 0 -> xyz=0.09 -0.12514 -0.0092692 rpy=0 0 0
